Commit message: added launch files

File: urdf/model.xacro (robot description, xacro)
@@ -41,5 +41,15 @@
   </inertial>
 </xacro:macro>
-<link name="base_link"/>
+<link name="base_footprint"/>
+<link name="base_link">
+   <xacro:default_visual    x_k ="${link_width}" y_k ="${link_width}" z_k ="${link_width}" x_c = "0." y_c = "0." z_c = "${link_length}"/>
+   <xacro:default_collision x_k ="${link_width}" y_k ="${link_width}" z_k ="${link_width}" x_c = "0." y_c = "0." z_c = "${link_length}"/>
+   <xacro:default_inertial  x_k ="${link_width}" y_k ="${link_width}" z_k ="${link_width}" x_c = "0." y_c = "0." z_c = "${link_length}" mass="${link_mass}"/>
+</link>
+<joint name="base_footprint_joint" type="fixed">
+  <parent link="base_footprint"/>
+  <child link="base_link"/>
+  <origin xyz="0 0 0" rpy="0 0 0"/>
+</joint>
 <!-- LINK: link1 -->
 <link name="link1">
@@ -74,5 +84,5 @@
   <parent link="link2"/>
   <child link="link3"/>
-  <origin xyz="0 0 ${link_length}" rpy="0 ${-PI/2} 0"/>
+  <origin xyz="0 0 ${link_length}" rpy="0 0 0"/>
   <axis xyz = "0 1 0"/>
 </joint>
@@ -99,3 +109,53 @@
   <axis xyz = "1 0 0"/>
 </joint>
+<transmission name="tran1">
+  <type>transmission_interface/SimpleTransmission</type>
+  <joint name="base_to_link1">
+    <hardwareInterface>hardware_interface/EffortJointInterface</hardwareInterface>
+  </joint>
+  <actuator name="motor1">
+    <hardwareInterface>hardware_interface/EffortJointInterface</hardwareInterface>
+    <mechanicalReduction>1</mechanicalReduction>
+  </actuator>
+</transmission>
+<transmission name="tran2">
+  <type>transmission_interface/SimpleTransmission</type>
+  <joint name="link1_to_link2">
+    <hardwareInterface>hardware_interface/EffortJointInterface</hardwareInterface>
+  </joint>
+  <actuator name="motor2">
+    <hardwareInterface>hardware_interface/EffortJointInterface</hardwareInterface>
+    <mechanicalReduction>1</mechanicalReduction>
+  </actuator>
+</transmission>
+<transmission name="tran3">
+  <type>transmission_interface/SimpleTransmission</type>
+  <joint name="link2_to_link3">
+    <hardwareInterface>hardware_interface/EffortJointInterface</hardwareInterface>
+  </joint>
+  <actuator name="motor3">
+    <hardwareInterface>hardware_interface/EffortJointInterface</hardwareInterface>
+    <mechanicalReduction>1</mechanicalReduction>
+  </actuator>
+</transmission>
+<transmission name="tran4">
+  <type>transmission_interface/SimpleTransmission</type>
+  <joint name="link3_to_link4">
+    <hardwareInterface>hardware_interface/EffortJointInterface</hardwareInterface>
+  </joint>
+  <actuator name="motor4">
+    <hardwareInterface>hardware_interface/EffortJointInterface</hardwareInterface>
+    <mechanicalReduction>1</mechanicalReduction>
+  </actuator>
+</transmission>
+<transmission name="tran5">
+  <type>transmission_interface/SimpleTransmission</type>
+  <joint name="link4_to_link5">
+    <hardwareInterface>hardware_interface/EffortJointInterface</hardwareInterface>
+  </joint>
+  <actuator name="motor5">
+    <hardwareInterface>hardware_interface/EffortJointInterface</hardwareInterface>
+    <mechanicalReduction>1</mechanicalReduction>
+  </actuator>
+</transmission>
 </robot>

Commit message: added damping

File: urdf/model.xacro (robot description, xacro)
@@ -64,4 +64,5 @@
   <origin xyz="0 0 0" rpy="0 0 0"/>
   <axis xyz = "0 0 1"/>
+  <dynamics damping="0.7"/>
 </joint>
 <link name="link2">
@@ -75,4 +76,5 @@
   <origin xyz="0 0 ${link_length}" rpy="0 0 0"/>
   <axis xyz = "0 1 0"/>
+  <dynamics damping="0.7"/>
 </joint>
 <link name="link3">
@@ -86,4 +88,5 @@
   <origin xyz="0 0 ${link_length}" rpy="0 0 0"/>
   <axis xyz = "0 1 0"/>
+  <dynamics damping="0.7"/>
 </joint>
 <link name="link4">
@@ -97,4 +100,5 @@
   <origin xyz="0 0 ${link_length}" rpy="0 0 0"/>
   <axis xyz = "0 1 0"/>
+  <dynamics damping="0.7"/>
 </joint>
 <link name="link5">
@@ -108,4 +112,5 @@
   <origin xyz="0 0 ${link_length}" rpy="0 0 0"/>
   <axis xyz = "1 0 0"/>
+  <dynamics damping="0.7"/>
 </joint>
 <transmission name="tran1">

Commit message: altered pid

File: urdf/model.xacro (robot description, xacro)
@@ -12,4 +12,6 @@
 <xacro:property name="link_length" value="0.2"/>
 <xacro:property name="link_width" value="0.05"/>
+<xacro:property name="base_width" value="1"/>
+<xacro:property name="base_height" value="0.2"/>
 <xacro:property name="link_mass" value="${density * link_width * link_width * link_length}"/>
 <xacro:macro name="default_visual" params = "x_k y_k z_k x_c y_c z_c">
@@ -43,7 +45,7 @@
 <link name="base_footprint"/>
 <link name="base_link">
-   <xacro:default_visual    x_k ="${link_width}" y_k ="${link_width}" z_k ="${link_width}" x_c = "0." y_c = "0." z_c = "${link_length}"/>
-   <xacro:default_collision x_k ="${link_width}" y_k ="${link_width}" z_k ="${link_width}" x_c = "0." y_c = "0." z_c = "${link_length}"/>
-   <xacro:default_inertial  x_k ="${link_width}" y_k ="${link_width}" z_k ="${link_width}" x_c = "0." y_c = "0." z_c = "${link_length}" mass="${link_mass}"/>
+   <xacro:default_visual    x_k ="${base_width}" y_k ="${base_width}" z_k ="${base_height}" x_c = "0." y_c = "0." z_c = "${base_height}"/>
+   <xacro:default_collision x_k ="${base_width}" y_k ="${base_width}" z_k ="${base_height}" x_c = "0." y_c = "0." z_c = "${base_height}"/>
+   <xacro:default_inertial  x_k ="${base_width}" y_k ="${base_width}" z_k ="${base_height}" x_c = "0." y_c = "0." z_c = "${base_height}" mass="${link_mass}"/>
 </link>
 <joint name="base_footprint_joint" type="fixed">
@@ -62,7 +64,7 @@
   <parent link="base_link"/>
   <child link="link1"/>
-  <origin xyz="0 0 0" rpy="0 0 0"/>
+  <origin xyz="0 0 ${base_height}" rpy="0 0 0"/>
   <axis xyz = "0 0 1"/>
-  <dynamics damping="0.7"/>
+    <dynamics damping="0.06"/>
 </joint>
 <link name="link2">
@@ -71,10 +73,11 @@
    <xacro:default_inertial  x_k ="${link_width}" y_k ="${link_width}" z_k ="${link_length}" x_c = "0." y_c = "0." z_c = "${link_length}" mass="${link_mass}"/>
 </link>
-<joint name="link1_to_link2" type="continuous">
+<joint name="link1_to_link2" type="revolute">
   <parent link="link1"/>
   <child link="link2"/>
   <origin xyz="0 0 ${link_length}" rpy="0 0 0"/>
   <axis xyz = "0 1 0"/>
-  <dynamics damping="0.7"/>
+  <limit effort="30" upper="1.5" lower="-1.5" velocity="1.0"/>
+    <dynamics damping="0.06"/>
 </joint>
 <link name="link3">
@@ -83,10 +86,10 @@
    <xacro:default_inertial  x_k ="${link_width}" y_k ="${link_width}" z_k ="${link_length}" x_c = "0." y_c = "0." z_c = "${link_length}" mass="${link_mass}"/>
 </link>
-<joint name="link2_to_link3" type="continuous">
+<joint name="link2_to_link3" type="revolute">
   <parent link="link2"/>
   <child link="link3"/>
   <origin xyz="0 0 ${link_length}" rpy="0 0 0"/>
   <axis xyz = "0 1 0"/>
-  <dynamics damping="0.7"/>
+  <limit effort="30" upper="1.5" lower="-1.5" velocity="1.0"/>
 </joint>
 <link name="link4">
@@ -95,10 +98,10 @@
    <xacro:default_inertial  x_k ="${link_width}" y_k ="${link_width}" z_k ="${link_length}" x_c = "0." y_c = "0." z_c = "${link_length}" mass="${link_mass}"/>
 </link>
-<joint name="link3_to_link4" type="continuous">
+<joint name="link3_to_link4" type="revolute">
   <parent link="link3"/>
   <child link="link4"/>
   <origin xyz="0 0 ${link_length}" rpy="0 0 0"/>
   <axis xyz = "0 1 0"/>
-  <dynamics damping="0.7"/>
+  <limit effort="30" upper="1.5" lower="-1.5" velocity="1.0"/>
 </joint>
 <link name="link5">
@@ -107,10 +110,11 @@
    <xacro:default_inertial  x_k ="${link_width}" y_k ="${link_width}" z_k ="${link_length}" x_c = "0." y_c = "0." z_c = "${link_length}" mass="${link_mass}"/>
 </link>
-<joint name="link4_to_link5" type="continuous">
+<joint name="link4_to_link5" type="revolute">
   <parent link="link4"/>
   <child link="link5"/>
   <origin xyz="0 0 ${link_length}" rpy="0 0 0"/>
   <axis xyz = "1 0 0"/>
-  <dynamics damping="0.7"/>
+  <limit effort="30" upper="1.5" lower="-1.5" velocity="1.0"/>
+  <dynamics damping="0.06"/>
 </joint>
 <transmission name="tran1">

Commit message: added controller

File: urdf/model.xacro (robot description, xacro)
@@ -69,52 +69,54 @@
 </joint>
 <link name="link2">
-   <xacro:default_visual    x_k ="${link_width}" y_k ="${link_width}" z_k ="${link_length}" x_c = "0." y_c = "0." z_c = "${link_length}"/>
-   <xacro:default_collision x_k ="${link_width}" y_k ="${link_width}" z_k ="${link_length}" x_c = "0." y_c = "0." z_c = "${link_length}"/>
-   <xacro:default_inertial  x_k ="${link_width}" y_k ="${link_width}" z_k ="${link_length}" x_c = "0." y_c = "0." z_c = "${link_length}" mass="${link_mass}"/>
+   <xacro:default_visual    x_k ="${link_width}" y_k ="${link_length}" z_k ="${link_width}" x_c = "0." y_c = "${link_length}" z_c = "${link_width}"/>
+   <xacro:default_collision x_k ="${link_width}" y_k ="${link_length}" z_k ="${link_width}" x_c = "0." y_c = "${link_length}" z_c = "${link_width}"/>
+   <xacro:default_inertial  x_k ="${link_width}" y_k ="${link_length}" z_k ="${link_width}" x_c = "0." y_c = "${link_length}" z_c = "${link_width}" mass="${link_mass}"/>
 </link>
 <joint name="link1_to_link2" type="revolute">
   <parent link="link1"/>
   <child link="link2"/>
-  <origin xyz="0 0 ${link_length}" rpy="0 0 0"/>
-  <axis xyz = "0 1 0"/>
+  <origin xyz="0 0 ${link_length}" rpy="${PI/2} 0 0"/>
+  <axis xyz = "0 0 1"/>
   <limit effort="30" upper="1.5" lower="-1.5" velocity="1.0"/>
     <dynamics damping="0.06"/>
 </joint>
 <link name="link3">
-   <xacro:default_visual    x_k ="${link_width}" y_k ="${link_width}" z_k ="${link_length}" x_c = "0." y_c = "0." z_c = "${link_length}"/>
-   <xacro:default_collision x_k ="${link_width}" y_k ="${link_width}" z_k ="${link_length}" x_c = "0." y_c = "0." z_c = "${link_length}"/>
-   <xacro:default_inertial  x_k ="${link_width}" y_k ="${link_width}" z_k ="${link_length}" x_c = "0." y_c = "0." z_c = "${link_length}" mass="${link_mass}"/>
+   <xacro:default_visual    x_k ="${link_width}" y_k ="${link_length}" z_k ="${link_width}" x_c = "0." y_c = "${link_length}" z_c = "${link_width}"/>
+   <xacro:default_collision x_k ="${link_width}" y_k ="${link_length}" z_k ="${link_width}" x_c = "0." y_c = "${link_length}" z_c = "${link_width}"/>
+   <xacro:default_inertial  x_k ="${link_width}" y_k ="${link_length}" z_k ="${link_width}" x_c = "0." y_c = "${link_length}" z_c = "${link_width}" mass="${link_mass}"/>
 </link>
 <joint name="link2_to_link3" type="revolute">
   <parent link="link2"/>
   <child link="link3"/>
-  <origin xyz="0 0 ${link_length}" rpy="0 0 0"/>
-  <axis xyz = "0 1 0"/>
+  <origin xyz="0 ${link_length} 0" rpy="0 0 0"/>
+  <axis xyz = "0 0 1"/>
   <limit effort="30" upper="1.5" lower="-1.5" velocity="1.0"/>
+    <dynamics damping="0.06"/>
 </joint>
 <link name="link4">
-   <xacro:default_visual    x_k ="${link_width}" y_k ="${link_width}" z_k ="${link_length}" x_c = "0." y_c = "0." z_c = "${link_length}"/>
-   <xacro:default_collision x_k ="${link_width}" y_k ="${link_width}" z_k ="${link_length}" x_c = "0." y_c = "0." z_c = "${link_length}"/>
-   <xacro:default_inertial  x_k ="${link_width}" y_k ="${link_width}" z_k ="${link_length}" x_c = "0." y_c = "0." z_c = "${link_length}" mass="${link_mass}"/>
+   <xacro:default_visual    x_k ="${link_width}" y_k ="${link_length}" z_k ="${link_width}" x_c = "0." y_c = "${link_length}" z_c = "${link_width}"/>
+   <xacro:default_collision x_k ="${link_width}" y_k ="${link_length}" z_k ="${link_width}" x_c = "0." y_c = "${link_length}" z_c = "${link_width}"/>
+   <xacro:default_inertial  x_k ="${link_width}" y_k ="${link_length}" z_k ="${link_width}" x_c = "0." y_c = "${link_length}" z_c = "${link_width}" mass="${link_mass}"/>
 </link>
 <joint name="link3_to_link4" type="revolute">
   <parent link="link3"/>
   <child link="link4"/>
-  <origin xyz="0 0 ${link_length}" rpy="0 0 0"/>
-  <axis xyz = "0 1 0"/>
+  <origin xyz="0 ${link_length} 0" rpy="0 0 0"/>
+  <axis xyz = "0 0 1"/>
   <limit effort="30" upper="1.5" lower="-1.5" velocity="1.0"/>
+    <dynamics damping="0.06"/>
 </joint>
 <link name="link5">
-   <xacro:default_visual    x_k ="${link_width}" y_k ="${link_width}" z_k ="${link_length}" x_c = "0." y_c = "0." z_c = "${link_length}"/>
-   <xacro:default_collision x_k ="${link_width}" y_k ="${link_width}" z_k ="${link_length}" x_c = "0." y_c = "0." z_c = "${link_length}"/>
-   <xacro:default_inertial  x_k ="${link_width}" y_k ="${link_width}" z_k ="${link_length}" x_c = "0." y_c = "0." z_c = "${link_length}" mass="${link_mass}"/>
+   <xacro:default_visual    x_k ="${link_width}" y_k ="${link_length}" z_k ="${link_width}" x_c = "0." y_c = "${link_length}" z_c = "${link_width}"/>
+   <xacro:default_collision x_k ="${link_width}" y_k ="${link_length}" z_k ="${link_width}" x_c = "0." y_c = "${link_length}" z_c = "${link_width}"/>
+   <xacro:default_inertial  x_k ="${link_width}" y_k ="${link_length}" z_k ="${link_width}" x_c = "0." y_c = "${link_length}" z_c = "${link_width}" mass="${link_mass}"/>
 </link>
 <joint name="link4_to_link5" type="revolute">
   <parent link="link4"/>
   <child link="link5"/>
-  <origin xyz="0 0 ${link_length}" rpy="0 0 0"/>
-  <axis xyz = "1 0 0"/>
+  <origin xyz="0 ${link_length} 0" rpy="0 ${PI/2} 0"/>
+  <axis xyz = "0 0 1"/>
   <limit effort="30" upper="1.5" lower="-1.5" velocity="1.0"/>
-  <dynamics damping="0.06"/>
+    <dynamics damping="0.06"/>
 </joint>
 <transmission name="tran1">
